File: WS2812ControllerEthernet.kicad_pcb (KiCad board)
At the start: 2 copper layers, 26.9 x 48.8 mm, 8 parts, among them J1 Conn_01x04_Male, J2 Conn_01x03_Male, J3 Conn_01x04_Male, U1 WT32_ETH01

Commit message: Work in Progress
Parts:
- moved J3 0.71 mm to (142.8, 105.6)
Connections:
- net Net-(J2-Pad2) renamed /DATA
- net Net-(J3-Pad2) renamed /TX
- net Net-(J3-Pad3) renamed /RX
Routing:
- net GPIO2: track 34.4 -> 0.00 mm
- net +5V: track 39.4 -> 8.39 mm
- net /DATA: track 5.40 -> 0.00 mm
Other:
- board text added: "D"
- board text added: "Power Supply"
- board text added: "VCC"

Commit message: First release, ready to order
Parts:
- removed the G*** at (146.6, 92.0)
- added F1: Fuse, halibs:Fuse-PTF75_Stelvio, B.Cu at (146.6, 61.3)
- added G***: LOGO, halibs:meintechblog, F.Cu at (146.7, 96.1)
- added G***: LOGO, halibs:Logo, F.Cu at (146.6, 89.2)
- added J4: Conn_01x02_Male, Connector_PinHeader_2.54mm:PinHeader_1x02_P2.54mm_Vertical, F.Cu at (153.8, 75.3)
- moved J1 10.6 mm to (136.4, 57.2)
- moved J2 9.80 mm to (151.6, 57.2)
- moved R1 5.47 mm to (150.2, 76.4)
Connections:
- net Net-(F1-Pad2) renamed /SUPPLY
- U1 pad 16: Net-(U1-Pad16) -> IO0
Routing:
- net +5V: track 8.39 -> 63.5 mm
- net GPIO2: track 0.00 -> 33.3 mm
- net /DATA: track 0.00 -> 19.8 mm
- net /SUPPLY: track 0.00 -> 11.5 mm
- net IO0: track 0.00 -> 8.45 mm
Other:
- board size 26.9 x 48.8 mm -> 26.9 x 59.8 mm
- net class Fet: trace_width 0.5 -> 1
- board text added: "5V"
- board text added: "FLASH"
- board text added: "Max. 6A !"
- board text added: "RX"
- board text added: "TX"

Commit message: Fixed wrong label
Parts:
- moved R1 10.8 mm to (139.4, 75.6)
- moved C1 5.59 mm to (148.5, 75.7)
Routing:
- net +5V: track 63.5 -> 84.6 mm
- net /SUPPLY: track 11.5 -> 22.7 mm
- net /DATA: track 19.8 -> 25.3 mm
- net GPIO2: track 33.3 -> 38.6 mm
Other:
- board text added: "v0.2"
- board text removed: "v0.1"
