File: WS2812ControllerEthernet.kicad_pcb (KiCad board)
At the start: 2 copper layers, 26.9 x 73.9 mm, 12 parts, among them J1 Barrel_Jack_MountingPin, J2 Conn_01x03_Pin, J3 Conn_01x03_Pin, J4 Conn_01x04_Male, J5 Conn_01x02_Male, U1 WT32_ETH01, U2 SN74AHCT125

Commit message: Update
Routing:
- net +5V: track 113.4 -> 128.8 mm
Other:
- board text added: "v2.1"
- board text removed: "v2.0"
Changed lines of the file:
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@@
 	(title_block
 		(title "WS2812-Controller Ethernet")
-		(date "2024-08-23")
+		(date "2024-08-27")
 		(rev "2.0")
 		(company "haus-automatisierung.com")
@@
 	)
 	(gr_line
-		(start 132.334 67.945)
-		(end 160.782 67.945)
+		(start 133.625541 71.245)
+		(end 159.490001 71.245)
 		(stroke
 			(width 0.12)
-			(type dash_dot)
+			(type dash_dot_dot)
+		)
+		(layer "B.SilkS")
+	)
+	(gr_line
+		(start 133.625541 67.945)
+		(end 159.490001 67.945)
+		(stroke
+			(width 0.12)
+			(type dash_dot_dot)
 		)
 		(layer "B.SilkS")
@@
 		)
 	)
-	(gr_text "v2.0"
+	(gr_text "v2.1"
 		(at 151.875 106.675 0)
 		(layer "F.SilkS")
@@
 	)
 	(segment
+		(start 140.525 75.910001)
+		(end 141.595 76.980001)
+		(width 1.5)
+		(layer "B.Cu")
+		(net 1)
+	)
+	(segment
 		(start 138.9395 51.756999)
 		(end 139.060001 51.8775)
@@
 		(width 1.5)
 		(layer "B.Cu")
+		(net 1)
+	)
+	(segment
+		(start 140.525 62)
+		(end 140.525 75.910001)
+		(width 1.5)
+		(layer "B.Cu")
